File: MCU Datalogger.kicad_sch (KiCad schematic)
At the start: 25 parts, among them U1 24LC1025, U2 24LC1025, U3 ATMEGA328P-AU, U4 DS1337S_, Y1 32.768kHz, Y2 16KHz

Commit message: fixed two bugs on the schematic related to the clock wiring
Connections:
- net SCK: no longer U1.6 (SCL), U2.6 (SCL), U3.28 (PC5), U4.6 (SCL)
- new net SCL: U1.6 (SCL), U2.6 (SCL), U3.28 (PC5), U4.6 (SCL)
Other:
- sheet Connectors ports: added SCL; removed none
Changed lines of the file:
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@@
 	(wire
 		(pts
+			(xy 207.01 142.24) (xy 214.63 142.24)
+		)
+		(stroke
+			(width 0)
+			(type default)
+		)
+	)
+	(wire
+		(pts
 			(xy 177.8 147.32) (xy 189.23 147.32)
 		)
@@
 	(wire
 		(pts
-			(xy 236.22 40.64) (xy 236.22 35.56)
+			(xy 180.34 143.51) (xy 189.23 143.51)
 		)
 		(stroke
@@
 	(wire
 		(pts
-			(xy 245.11 29.21) (xy 245.11 35.56)
+			(xy 236.22 40.64) (xy 236.22 35.56)
 		)
 		(stroke
@@
 	(wire
 		(pts
-			(xy 180.34 130.81) (xy 189.23 130.81)
+			(xy 180.34 140.97) (xy 189.23 140.97)
 		)
 		(stroke
@@
 		)
 	)
-	(wire
-		(pts
-			(xy 180.34 138.43) (xy 189.23 138.43)
-		)
-		(stroke
-			(width 0)
-			(type default)
-		)
-	)
 	(rectangle
 		(start 254 113.03)
@@
 		)
 	)
-	(label "SCK"
-		(at 180.34 138.43 180)
+	(label "MISO"
+		(at 214.63 147.32 0)
 		(fields_autoplaced yes)
 		(effects
@@
 				(size 1.27 1.27)
 			)
-			(justify right bottom)
+			(justify left bottom)
 		)
 	)
-	(label "MISO"
-		(at 214.63 147.32 0)
+	(label "D7"
+		(at 231.14 60.96 0)
 		(fields_autoplaced yes)
 		(effects
@@
 		)
 	)
-	(label "SCK"
-		(at 52.07 63.5 0)
+	(label "SCL"
+		(at 180.34 143.51 180)
 		(fields_autoplaced yes)
 		(effects
@@
 				(size 1.27 1.27)
 			)
-			(justify left bottom)
+			(justify right bottom)
 		)
 	)
-	(label "D7"
-		(at 231.14 60.96 0)
+	(label "D3"
+		(at 210.82 121.92 0)
 		(fields_autoplaced yes)
 		(effects
@@
 		)
 	)
-	(label "D3"
-		(at 210.82 121.92 0)
+	(label "SCL"
+		(at 62.23 157.48 0)
 		(fields_autoplaced yes)
 		(effects
@@
 		)
 	)
+	(label "SCL"
+		(at 102.87 157.48 0)
+		(fields_autoplaced yes)
+		(effects
+			(font
+				(size 1.27 1.27)
+			)
+			(justify left bottom)
+		)
+	)
 	(label "Vcc"
 		(at 82.55 160.02 180)
@@
 	)
 	(label "SDA"
-		(at 180.34 130.81 180)
+		(at 180.34 140.97 180)
 		(fields_autoplaced yes)
 		(effects
@@
 		)
 	)
-	(label "SCK"
+	(label "SCL"
 		(at 200.66 78.74 180)
 		(fields_autoplaced yes)
@@
 		)
 	)
+	(label "SCK"
+		(at 214.63 142.24 0)
+		(fields_autoplaced yes)
+		(effects
+			(font
+				(size 1.27 1.27)
+			)
+			(justify left bottom)
+		)
+	)
 	(label "D4"
 		(at 210.82 124.46 0)
@@
 		)
 	)
+	(label "SCL"
+		(at 52.07 63.5 180)
+		(fields_autoplaced yes)
+		(effects
+			(font
+				(size 1.27 1.27)
+			)
+			(justify right bottom)
+		)
+	)
 	(label "RESET"
 		(at 214.63 153.67 0)
@@
 	)
 	(label "SDA"
-		(at 52.07 71.12 0)
+		(at 52.07 71.12 180)
 		(fields_autoplaced yes)
 		(effects
@@
 				(size 1.27 1.27)
 			)
-			(justify left bottom)
+			(justify right bottom)
 		)
 	)
@@
 		)
 	)
-	(label "SCK"
-		(at 102.87 157.48 0)
-		(fields_autoplaced yes)
-		(effects
-			(font
-				(size 1.27 1.27)
-			)
-			(justify left bottom)
-		)
-	)
-	(label "SCK"
-		(at 62.23 157.48 0)
-		(fields_autoplaced yes)
-		(effects
-			(font
-				(size 1.27 1.27)
-			)
-			(justify left bottom)
-		)
-	)
 	(label "RX"
 		(at 177.8 147.32 180)
@@
 	)
 	(symbol
-		(lib_id "power:PWR_FLAG")
-		(at 245.11 29.21 0)
-		(unit 1)
-		(exclude_from_sim no)
-		(in_bom yes)
-		(on_board yes)
-		(dnp no)
-		(fields_autoplaced yes)
-		(property "Reference" "#FLG01"
-			(at 245.11 27.305 0)
-			(effects
-				(font
-					(size 1.27 1.27)
-				)
-				(hide yes)
-			)
-		)
-		(property "Value" "PWR_FLAG"
-			(at 245.11 24.13 0)
-			(effects
-				(font
-					(size 1.27 1.27)
-				)
-			)
-		)
-		(property "Footprint" ""
-			(at 245.11 29.21 0)
-			(effects
-				(font
-					(size 1.27 1.27)
-				)
-				(hide yes)
-			)
-		)
-		(property "Datasheet" "~"
-			(at 245.11 29.21 0)
-			(effects
-				(font
-					(size 1.27 1.27)
-				)
-				(hide yes)
-			)
-		)
-		(property "Description" "Special symbol for telling ERC where power comes from"
-			(at 245.11 29.21 0)
-			(effects
-				(font
-					(size 1.27 1.27)
-				)
-				(hide yes)
-			)
-		)
-		(pin "1"
-		)
-		(instances
-			(project ""
-				(path "/2d095fec-de04-4caa-8a5d-d4c981edd86b"
-					(reference "#FLG01")
-					(unit 1)
-				)
-			)
-		)
-	)
-	(symbol
 		(lib_id "Memory_EEPROM:24LC1025")
 		(at 92.71 157.48 0)
@@
 			)
 		)
-		(pin "SCK" passive
-			(at 189.23 138.43 180)
-			(effects
-				(font
-					(size 1.27 1.27)
-				)
-				(justify left)
-			)
-		)
 		(pin "GND" passive
 			(at 189.23 119.38 180)
@@
 		)
 		(pin "SDA" bidirectional
-			(at 189.23 130.81 180)
+			(at 189.23 140.97 180)
 			(effects
 				(font
@@
 			(effects
 				(font
+					(size 1.27 1.27)
+				)
+				(justify right)
+			)
+		)
+		(pin "SCL" passive
+			(at 189.23 143.51 180)
+			(effects
+				(font
+					(size 1.27 1.27)
+				)
+				(justify left)
+			)
+		)
+		(pin "SCK" passive
+			(at 207.01 142.24 0)
+			(effects
+				(font

Commit message: finished an improved version of the 2 layer PCB
Connections:
- net SCK: no longer R3.2
- net SCL: now also R3.2
Changed lines of the file:
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@@
 		)
 	)
-	(label "SCK"
+	(label "SCL"
 		(at 118.11 165.1 0)
 		(fields_autoplaced yes)
